File: board_design/PCB/_autosave-Final TP.sch (KiCad schematic (older format))
At the start: 14 parts, among them SW1 Reset

Commit message: uploaded folders
Parts:
- added R4, R5: R, symbol Device:R
- renumbered Power to Power1
Connections:
- net +9V: now also R4.1
- net Earth: now also R5.2
- net at HC-5.4 (Pin_4): now also R4.2, R5.1
Changed lines of the file:
@@
 $EndComp
 $Comp
-L Connector_Generic:Conn_01x02 Power
+L Connector_Generic:Conn_01x02 Power1
 U 1 1 5D74B06D
 P 2850 2600
-F 0 "Power" H 2850 2350 50  0000 C CNN
+F 0 "Power1" H 2850 2350 50  0000 C CNN
 F 1 "GND" H 2850 2750 50  0000 C CNN
 F 2 "" H 2850 2600 50  0001 C CNN
@@
 Wire Wire Line
 	5600 3250 5600 3400
-Text Notes 6100 2450 0    50   ~ 0
-5V
 $Comp
 L power:Earth #PWR01
@@
 	3400 2200 3400 2100
 $Comp
-L power:+9V #PWR?
+L power:+9V #PWR05
 U 1 1 5D768167
 P 3050 2150
-F 0 "#PWR?" H 3050 2000 50  0001 C CNN
+F 0 "#PWR05" H 3050 2000 50  0001 C CNN
 F 1 "+9V" H 3000 2300 50  0000 C CNN
 F 2 "" H 3050 2150 50  0001 C CNN
@@
 	3950 2200 3950 1950
 $Comp
-L power:Earth #PWR?
+L power:Earth #PWR09
 U 1 1 5D77BCA8
 P 3950 3500
-F 0 "#PWR?" H 3950 3250 50  0001 C CNN
+F 0 "#PWR09" H 3950 3250 50  0001 C CNN
 F 1 "Earth" H 3950 3350 50  0001 C CNN
 F 2 "" H 3950 3500 50  0001 C CNN
@@
 	3950 2600 4450 2600
 $Comp
-L power:+9V #PWR?
+L power:+9V #PWR08
 U 1 1 5D78E7B6
 P 3950 1950
-F 0 "#PWR?" H 3950 1800 50  0001 C CNN
+F 0 "#PWR08" H 3950 1800 50  0001 C CNN
 F 1 "+9V" H 3965 2123 50  0000 C CNN
 F 2 "" H 3950 1950 50  0001 C CNN
@@
 $EndComp
 $Comp
-L power:Earth #PWR?
+L power:Earth #PWR06
 U 1 1 5D78F0E6
 P 3050 2800
-F 0 "#PWR?" H 3050 2550 50  0001 C CNN
+F 0 "#PWR06" H 3050 2550 50  0001 C CNN
 F 1 "Earth" H 3050 2650 50  0001 C CNN
 F 2 "" H 3050 2800 50  0001 C CNN
@@
 	3400 3400 3400 3500
 $Comp
-L power:Earth #PWR?
+L power:Earth #PWR07
 U 1 1 5D792B65
 P 3400 3500
-F 0 "#PWR?" H 3400 3250 50  0001 C CNN
+F 0 "#PWR07" H 3400 3250 50  0001 C CNN
 F 1 "Earth" H 3400 3350 50  0001 C CNN
 F 2 "" H 3400 3500 50  0001 C CNN
@@
 $EndComp
 $Comp
-L power:Earth #PWR?
+L power:Earth #PWR010
 U 1 1 5D7951CF
 P 5600 3950
-F 0 "#PWR?" H 5600 3700 50  0001 C CNN
+F 0 "#PWR010" H 5600 3700 50  0001 C CNN
 F 1 "Earth" H 5600 3800 50  0001 C CNN
 F 2 "" H 5600 3950 50  0001 C CNN
@@
 $EndComp
 $Comp
-L power:Earth #PWR?
+L power:Earth #PWR011
 U 1 1 5D796651
 P 5900 3950
-F 0 "#PWR?" H 5900 3700 50  0001 C CNN
+F 0 "#PWR011" H 5900 3700 50  0001 C CNN
 F 1 "Earth" H 5900 3800 50  0001 C CNN
 F 2 "" H 5900 3950 50  0001 C CNN
@@
 	1    0    0    -1
 $EndComp
-$Comp
-L power:Earth #PWR05
-U 1 1 5D7FB6B0
-P 5950 2350
-F 0 "#PWR05" H 5950 2100 50  0001 C CNN
-F 1 "Earth" H 5950 2200 50  0001 C CNN
-F 2 "" H 5950 2350 50  0001 C CNN
-F 3 "~" H 5950 2350 50  0001 C CNN
-	1    5950 2350
-	1    0    0    -1
-$EndComp
-Wire Wire Line
-	5950 2350 6150 2350
 Wire Wire Line
 	3400 3050 3400 3100
@@
 Wire Wire Line
 	5900 3950 5900 3650
+$Comp
+L Device:R R4
+U 1 1 5D7704F5
+P 5750 2200
+F 0 "R4" H 5650 2350 50  0000 L CNN
+F 1 "R" H 5650 2050 50  0000 L CNN
+F 2 "" V 5680 2200 50  0001 C CNN
+F 3 "~" H 5750 2200 50  0001 C CNN
+	1    5750 2200
+	1    0    0    -1
+$EndComp
+$Comp
+L Device:R R5
+U 1 1 5D770BA1
+P 5750 2750
+F 0 "R5" H 5650 2900 50  0000 L CNN
+F 1 "R" H 5650 2600 50  0000 L CNN
+F 2 "" V 5680 2750 50  0001 C CNN
+F 3 "~" H 5750 2750 50  0001 C CNN
+	1    5750 2750
+	1    0    0    -1
+$EndComp
+Wire Wire Line
+	5750 2050 5750 1950
+Text Notes 6100 2450 0    50   ~ 0
+5V
+Wire Wire Line
+	5750 2350 5750 2450
+Wire Wire Line
+	5750 2450 5750 2600
+Connection ~ 5750 2450
+Wire Wire Line
+	5750 2450 6150 2450
+Wire Wire Line
+	5950 2350 6150 2350
+Wire Wire Line
+	5950 2350 5950 2550
+$Comp
+L power:Earth #PWR012
+U 1 1 5D77EAEC
+P 5950 2550
+F 0 "#PWR012" H 5950 2300 50  0001 C CNN
+F 1 "Earth" H 5950 2400 50  0001 C CNN
+F 2 "" H 5950 2550 50  0001 C CNN
+F 3 "~" H 5950 2550 50  0001 C CNN
+	1    5950 2550
+	1    0    0    -1
+$EndComp
+$Comp
+L power:+9V #PWR?
+U 1 1 5D780D03
+P 5750 1950
+F 0 "#PWR?" H 5750 1800 50  0001 C CNN
+F 1 "+9V" H 5765 2123 50  0000 C CNN
+F 2 "" H 5750 1950 50  0001 C CNN
+F 3 "" H 5750 1950 50  0001 C CNN
+	1    5750 1950
+	1    0    0    -1
+$EndComp
+$Comp
+L power:Earth #PWR?
+U 1 1 5D7840E6
+P 5750 3050
+F 0 "#PWR?" H 5750 2800 50  0001 C CNN
+F 1 "Earth" H 5750 2900 50  0001 C CNN
+F 2 "" H 5750 3050 50  0001 C CNN
+F 3 "~" H 5750 3050 50  0001 C CNN
+	1    5750 3050
+	1    0    0    -1
+$EndComp
+Wire Wire Line
+	5750 3050 5750 2900
 $EndSCHEMATC

Commit message: update
Parts:
- removed R3: R, symbol Device:R
- C1, C2: footprint (none) -> Capacitor_THT:C_Disc_D4.3mm_W1.9mm_P5.00mm
- D1: footprint (none) -> LED_THT:LED_D3.0mm
- GasSensor1, HC-5, PiesoSpeaker1: footprint (none) -> Connector_PinHeader_2.54mm:PinHeader_1x03_P2.54mm_Horizontal
- Power1: footprint (none) -> Resistor_THT:R_Axial_DIN0207_L6.3mm_D2.5mm_P15.24mm_Horizontal
- R1: value R -> 2.8K; footprint (none) -> Resistor_THT:R_Axial_DIN0207_L6.3mm_D2.5mm_P15.24mm_Horizontal
- R2: value R -> 1.62K; footprint (none) -> Resistor_THT:R_Axial_DIN0207_L6.3mm_D2.5mm_P15.24mm_Horizontal
- R3: value R -> 2.8k; footprint (none) -> Resistor_THT:R_Axial_DIN0207_L6.3mm_D2.5mm_P15.24mm_Horizontal
- R4: value R -> 2.8k; footprint (none) -> Resistor_THT:R_Axial_DIN0207_L6.3mm_D2.5mm_P10.16mm_Horizontal
- R5: value R -> 1.62k; footprint (none) -> Resistor_THT:R_Axial_DIN0207_L6.3mm_D2.5mm_P5.08mm_Vertical
- SW1: footprint (none) -> Connector_PinHeader_2.54mm:PinHeader_1x03_P2.54mm_Vertical
- renumbered DIP28 to U1
Connections:
- net at U1.5 (PD3): now also PiesoSpeaker1.1 (Pin_1)
Other:
- moved on the sheet: R4, R5
Changed lines of the file:
@@
 $EndDescr
 $Comp
-L Final-TP-rescue:ATmega238-mylib DIP28
+L Final-TP-rescue:ATmega238-mylib U1
 U 1 1 5D74969E
 P 5000 2750
-F 0 "DIP28" H 4850 2000 79  0000 C CNN
-F 1 "ATmega238P" H 4850 3700 70  0000 C CNN
+F 0 "U1" H 4850 2050 79  0000 C CNN
+F 1 "ATmega238P" H 4900 3650 70  0000 C CNN
 F 2 "" H 4400 3050 50  0001 C CNN
 F 3 "" H 4400 3050 50  0001 C CNN
@@
 U 1 1 5D7508D0
 P 3950 2350
-F 0 "R1" H 3850 2500 50  0000 L CNN
-F 1 "R" H 3850 2200 50  0000 L CNN
-F 2 "" V 3880 2350 50  0001 C CNN
+F 0 "R1" H 3800 2500 50  0000 L CNN
+F 1 "2.8K" H 3750 2200 50  0000 L CNN
+F 2 "Resistor_THT:R_Axial_DIN0207_L6.3mm_D2.5mm_P15.24mm_Horizontal" V 3880 2350 50  0001 C CNN
 F 3 "~" H 3950 2350 50  0001 C CNN
 	1    3950 2350
@@
 U 1 1 5D74B06D
 P 2850 2600
-F 0 "Power1" H 2850 2350 50  0000 C CNN
-F 1 "GND" H 2850 2750 50  0000 C CNN
-F 2 "" H 2850 2600 50  0001 C CNN
+F 0 "Power1" H 2900 2400 50  0000 C CNN
+F 1 "GND" H 2950 2700 50  0000 C CNN
+F 2 "Resistor_THT:R_Axial_DIN0207_L6.3mm_D2.5mm_P15.24mm_Horizontal" H 2850 2600 50  0001 C CNN
 F 3 "~" H 2850 2600 50  0001 C CNN
 	1    2850 2600
 	-1   0    0    1
 $EndComp
-$Comp
-L Device:R R3
-U 1 1 5D764769
-P 4150 2100
-F 0 "R3" H 4050 2250 50  0000 L CNN
-F 1 "R" H 4050 1950 50  0000 L CNN
-F 2 "" V 4080 2100 50  0001 C CNN
-F 3 "~" H 4150 2100 50  0001 C CNN
-	1    4150 2100
-	1    0    0    -1
-$EndComp
 Text Notes 4300 2400 0    50   ~ 0
 PWM
@@
 U 1 1 5D761CF2
 P 6150 3550
-F 0 "PiesoSpeaker1" H 5950 3700 50  0000 L CNN
-F 1 "Conn_01x02" H 5950 3300 50  0000 L CNN
-F 2 "" H 6150 3550 50  0001 C CNN
+F 0 "PiesoSpeaker1" H 6000 3700 50  0000 L CNN
+F 1 "Conn_01x02" H 6050 3300 50  0000 L CNN
+F 2 "Connector_PinHeader_2.54mm:PinHeader_1x03_P2.54mm_Horizontal" H 6150 3550 50  0001 C CNN
 F 3 "~" H 6150 3550 50  0001 C CNN
 	1    6150 3550
@@
 U 1 1 5D75F460
 P 5600 3100
-F 0 "R3" H 5650 2950 40  0000 C CNN
-F 1 "R" H 5650 3250 50  0000 C CNN
-F 2 "" V 5530 3100 50  0001 C CNN
+F 0 "R3" H 5700 3000 40  0000 C CNN
+F 1 "2.8k" H 5700 3250 50  0000 C CNN
+F 2 "Resistor_THT:R_Axial_DIN0207_L6.3mm_D2.5mm_P15.24mm_Horizontal" V 5530 3100 50  0001 C CNN
 F 3 "~" H 5600 3100 50  0001 C CNN
 	1    5600 3100
@@
 U 1 1 5D75CF16
 P 5600 3550
-F 0 "D1" V 5700 3650 50  0000 C CNN
-F 1 "LED1" V 5450 3650 50  0000 C CNN
-F 2 "" H 5600 3550 50  0001 C CNN
+F 0 "D1" V 5650 3700 50  0000 C CNN
+F 1 "LED1" V 5500 3700 50  0000 C CNN
+F 2 "LED_THT:LED_D3.0mm" H 5600 3550 50  0001 C CNN
 F 3 "~" H 5600 3550 50  0001 C CNN
 	1    5600 3550
@@
 F 0 "HC-5" H 6250 2500 50  0000 L CNN
 F 1 "Conn_01x04" H 6150 1900 50  0000 L CNN
-F 2 "" H 6350 2250 50  0001 C CNN
+F 2 "Connector_PinHeader_2.54mm:PinHeader_1x03_P2.54mm_Horizontal" H 6350 2250 50  0001 C CNN
 F 3 "~" H 6350 2250 50  0001 C CNN
 	1    6350 2250
@@
 F 0 "C1" H 3250 2450 50  0000 L CNN
 F 1 "20pF" H 3200 2250 50  0000 L CNN
-F 2 "" H 3438 2200 50  0001 C CNN
+F 2 "Capacitor_THT:C_Disc_D4.3mm_W1.9mm_P5.00mm" H 3438 2200 50  0001 C CNN
 F 3 "~" H 3400 2350 50  0001 C CNN
 	1    3400 2350
@@
 F 0 "C2" H 3250 3350 50  0000 L CNN
 F 1 "20pF" H 3200 3150 50  0000 L CNN
-F 2 "" H 3438 3100 50  0001 C CNN
+F 2 "Capacitor_THT:C_Disc_D4.3mm_W1.9mm_P5.00mm" H 3438 3100 50  0001 C CNN
 F 3 "~" H 3400 3250 50  0001 C CNN
 	1    3400 3250
@@
 P 3400 1700
 F 0 "GasSensor1" H 3200 1350 50  0000 L CNN
-F 1 "Conn_01x06" H 3200 1900 50  0000 L CNN
-F 2 "" H 3400 1700 50  0001 C CNN
+F 1 "Conn_01x06" H 3200 1950 50  0000 L CNN
+F 2 "Connector_PinHeader_2.54mm:PinHeader_1x03_P2.54mm_Horizontal" H 3400 1700 50  0001 C CNN
 F 3 "~" H 3400 1700 50  0001 C CNN
 	1    3400 1700
@@
 Wire Wire Line
 	3600 1500 5350 1500
-Wire Wire Line
-	4150 2400 4150 2250
 Wire Wire Line
 	4150 2400 4450 2400
@@
 U 1 1 5D7850D8
 P 4650 1350
-F 0 "SW1" H 4650 1300 50  0000 C CNN
-F 1 "Reset" H 4650 1450 50  0000 C CNN
-F 2 "" H 4650 1550 50  0001 C CNN
+F 0 "SW1" H 4650 1250 50  0000 C CNN
+F 1 "Reset" H 4650 1550 50  0000 C CNN
+F 2 "Connector_PinHeader_2.54mm:PinHeader_1x03_P2.54mm_Vertical" H 4650 1550 50  0001 C CNN
 F 3 "~" H 4650 1550 50  0001 C CNN
 	1    4650 1350
@@
 U 1 1 5D7512B6
 P 3950 2850
-F 0 "R2" H 3850 2700 50  0000 L CNN
-F 1 "R" H 3850 3000 50  0000 L CNN
-F 2 "" V 3880 2850 50  0001 C CNN
+F 0 "R2" H 3800 2950 50  0000 L CNN
+F 1 "1.62K" H 3700 2750 50  0000 L CNN
+F 2 "Resistor_THT:R_Axial_DIN0207_L6.3mm_D2.5mm_P15.24mm_Horizontal" V 3880 2850 50  0001 C CNN
 F 3 "~" H 3950 2850 50  0001 C CNN
 	1    3950 2850
@@
 	3400 2650 4400 2650
 Wire Wire Line
-	4150 1600 4150 1950
-Wire Wire Line
 	4300 1650 4300 2200
 Wire Wire Line
@@
 L Device:R R4
 U 1 1 5D7704F5
-P 5750 2200
-F 0 "R4" H 5650 2350 50  0000 L CNN
-F 1 "R" H 5650 2050 50  0000 L CNN
-F 2 "" V 5680 2200 50  0001 C CNN
-F 3 "~" H 5750 2200 50  0001 C CNN
-	1    5750 2200
+P 5750 2100
+F 0 "R4" H 5600 2200 50  0000 L CNN
+F 1 "2.8k" H 5550 2000 50  0000 L CNN
+F 2 "Resistor_THT:R_Axial_DIN0207_L6.3mm_D2.5mm_P10.16mm_Horizontal" V 5680 2100 50  0001 C CNN
+F 3 "~" H 5750 2100 50  0001 C CNN
+	1    5750 2100
 	1    0    0    -1
 $EndComp
@@
 L Device:R R5
 U 1 1 5D770BA1
-P 5750 2750
-F 0 "R5" H 5650 2900 50  0000 L CNN
-F 1 "R" H 5650 2600 50  0000 L CNN
-F 2 "" V 5680 2750 50  0001 C CNN
-F 3 "~" H 5750 2750 50  0001 C CNN
-	1    5750 2750
-	1    0    0    -1
-$EndComp
-Wire Wire Line
-	5750 2050 5750 1950
-Text Notes 6100 2450 0    50   ~ 0
+P 5750 2700
+F 0 "R5" H 5600 2800 50  0000 L CNN
+F 1 "1.62k" H 5500 2600 50  0000 L CNN
+F 2 "Resistor_THT:R_Axial_DIN0207_L6.3mm_D2.5mm_P5.08mm_Vertical" V 5680 2700 50  0001 C CNN
+F 3 "~" H 5750 2700 50  0001 C CNN
+	1    5750 2700
+	1    0    0    -1
+$EndComp
+Text Notes 6050 2450 0    50   ~ 0
 5V
-Wire Wire Line
-	5750 2350 5750 2450
-Wire Wire Line
-	5750 2450 5750 2600
-Connection ~ 5750 2450
 Wire Wire Line
 	5750 2450 6150 2450
@@
 $EndComp
 $Comp
-L power:+9V #PWR?
-U 1 1 5D780D03
-P 5750 1950
-F 0 "#PWR?" H 5750 1800 50  0001 C CNN
-F 1 "+9V" H 5765 2123 50  0000 C CNN
-F 2 "" H 5750 1950 50  0001 C CNN
-F 3 "" H 5750 1950 50  0001 C CNN
-	1    5750 1950
-	1    0    0    -1
-$EndComp
-$Comp
-L power:Earth #PWR?
+L power:Earth #PWR014
 U 1 1 5D7840E6
 P 5750 3050
-F 0 "#PWR?" H 5750 2800 50  0001 C CNN
+F 0 "#PWR014" H 5750 2800 50  0001 C CNN
 F 1 "Earth" H 5750 2900 50  0001 C CNN
 F 2 "" H 5750 3050 50  0001 C CNN
@@
 	1    0    0    -1
 $EndComp
-Wire Wire Line
-	5750 3050 5750 2900
+$Comp
+L power:+9V #PWR013
+U 1 1 5D780D03
+P 5750 1900
+F 0 "#PWR013" H 5750 1750 50  0001 C CNN
+F 1 "+9V" H 5750 2050 50  0000 C CNN
+F 2 "" H 5750 1900 50  0001 C CNN
+F 3 "" H 5750 1900 50  0001 C CNN
+	1    5750 1900
+	1    0    0    -1
+$EndComp
+Wire Wire Line
+	5750 2250 5750 2450
+Wire Wire Line
+	5750 2850 5750 3050
+Wire Wire Line
+	4150 1600 4150 2400
+Wire Wire Line
+	5750 1900 5750 1950
+Wire Wire Line
+	5750 2550 5750 2450
+Connection ~ 5750 2450
 $EndSCHEMATC
